Commit message: test_merge

File: src/ls01b_v2/urdf/cona.urdf (robot description, URDF)
Before this commit: robot cona, 4 links, 3 joints
Links:
- removed link camera
- removed link lidar1
- removed link lidar2
- added link camera_link
- added link laser1
- added link laser2
Joints:
- joint robot2camera: child camera -> camera_link; origin xyz=0.2 0 0 rpy=0 0 4.71 -> xyz=0.15 0 0 rpy=0 0 4.71
- joint robot2laser1: child lidar1 -> laser1; origin xyz=0.2 0.2 0 rpy=0 0 0.785 -> xyz=0.15 0.105 0 rpy=0 0 0.785
- joint robot2laser2: child lidar2 -> laser2; origin xyz=-0.2 -0.2 0 rpy=0 0 3.925 -> xyz=-0.15 -0.105 0 rpy=0 0 3.925

Commit message: test

File: src/ls01b_v2/urdf/cona.urdf (robot description, URDF)
Before this commit: robot cona, 4 links, 3 joints
Links:
- added link laser3
Joints:
- added joint robot2laser3: type fixed, parent base_link, child laser3, origin xyz=0 0 0 rpy=0 0 0
